Commit message: Add new version of description

File: urdf/robokit_hardware.xacro (robot description, xacro)
@@ -1,11 +1,11 @@
 <?xml version="1.0"?>
 <robot xmlns:xacro="http://www.ros.org/wiki/xacro">
-  <xacro:macro name="robokit_ros2_control" params="port baud timeout">
+  <xacro:macro name="robokit_ros2_control" params="port baudrate timeout">
     <ros2_control name="RobokitHardware" type="system">
       <hardware>
-          <plugin>robokit_hardware/RobokitHardwareInterface</plugin>
-          <param name="port">     ${port}    </param>
-          <param name="baudrate"> ${baud}    </param>
-          <param name="timeout">  ${timeout} </param>
+          <plugin>robokit_hardware/RobokitHardware</plugin>
+          <param name="port">${port}</param>
+          <param name="baudrate">${baudrate}</param>
+          <param name="timeout">${timeout} </param>
       </hardware>
       <xacro:macro name="configure_joint" params="joint_name id sio">

File: urdf/robokit_hardware_new.xacro (robot description, xacro)
@@ -1,16 +1,18 @@
 <?xml version="1.0"?>
 <robot xmlns:xacro="http://www.ros.org/wiki/xacro">
-  <xacro:macro name="robokit_ros2_control" params="port baud timeout">
+  <xacro:macro name="robokit_ros2_control" params="port baudrate timeout">
     <ros2_control name="RobokitHardware" type="system">
       <hardware>
-          <plugin>robokit_hardware/RobokitHardwareInterface</plugin>
-          <param name="port">     ${port}    </param>
-          <param name="baudrate"> ${baud}    </param>
-          <param name="timeout">  ${timeout} </param>
+          <plugin>robokit_hardware/RobokitHardware</plugin>
+          <param name="port">${port}</param>
+          <param name="baudrate">${baudrate}</param>
+          <param name="timeout">${timeout} </param>
       </hardware>
+      <xacro:property name="config_path" value="$(env DESCRIPTION_PATH)/config/servos.yaml"/>
+      <xacro:property name="config" value="${load_yaml(config_path)}"/>
       <xacro:macro name="configure_joint" params="joint_name id sio">
         <joint name="${joint_name}">
-          <param name="id">  ${id}  </param>
-          <param name="sio"> ${sio} </param>
+          <param name="id">  ${config['${joint_name}']['id']} </param>
+          <param name="sio"> ${config['${joint_name}']['id']} </param>
           <command_interface name="position"/>
           <state_interface name="position"/>
@@ -42,4 +44,4 @@
     </ros2_control>
   </xacro:macro>
-  <xacro:robokit_ros2_control port="/dev/pts/1" baud="38400" timeout="1"/>
+  <xacro:robokit_ros2_control port="ppp" baudrate="bbb" timeout="ttt"/>
 </robot>

File: urdf/robokit_mv.urdf.xacro (robot description, xacro)
@@ -6,5 +6,5 @@
     <xacro:arg name="use_sim" default="true"/>
     <xacro:arg name="port"    default="none"/>
-    <xacro:arg name="baud"    default="none"/>
+    <xacro:arg name="baudrate"    default="none"/>
     <xacro:arg name="timeout" default="none"/>
     <!--> Hardware setup (webots or real) <!-->
@@ -14,5 +14,5 @@
     <xacro:unless value="$(arg use_sim)">
       <xacro:include filename="robokit_hardware.xacro"/>
-      <xacro:robokit_ros2_control port="$(arg port)" baud="$(arg baud)" timeout="$(arg timeout)"/>
+      <xacro:robokit_ros2_control port="$(arg port)" baudrate="$(arg baudrate)" timeout="$(arg timeout)"/>
     </xacro:unless>
     <link
